Commit message: 整体启动+机械臂描述部分启动

File: src/description/urdf/yam.urdf (robot description, URDF)
Before this commit: robot yam_v0, 7 links, 6 joints
Links:
- link base_link: geometry collision mesh filename=http://192.168.1.184:9091/meshes/base_link_collision.stl; visual mesh filename=http://192.168.1.184:9091/meshes/base_link_visual.stl
- link link_1: geometry collision mesh filename=http://192.168.1.184:9091/meshes/link_1_collision.stl; visual mesh filename=http://192.168.1.184:9091/meshes/link_1_visual.stl
- link link_2: geometry collision mesh filename=http://192.168.1.184:9091/meshes/link_2_collision.stl; visual mesh filename=http://192.168.1.184:9091/meshes/link_2_visual.stl
- link link_3: geometry collision mesh filename=http://192.168.1.184:9091/meshes/link_3_collision.stl; visual mesh filename=http://192.168.1.184:9091/meshes/link_3_visual.stl
- link link_4: geometry collision mesh filename=http://192.168.1.184:9091/meshes/link_4_collision.stl; visual mesh filename=http://192.168.1.184:9091/meshes/link_4_visual.stl
- link link_5: geometry collision mesh filename=http://192.168.1.184:9091/meshes/link_5_collision.stl; visual mesh filename=http://192.168.1.184:9091/meshes/link_5_visual.stl
- link link_6: geometry collision mesh filename=http://192.168.1.184:9091/meshes/link_6_collision.stl; visual mesh filename=http://192.168.1.184:9091/meshes/link_6_visual.stl
